File: RECESSIM-CW312T-SAM4C32.kicad_sch (KiCad schematic)
At the start: 102 parts, among them U1 ATSAM4C32C

Commit message: Finalized Rev1 of the PCB design, removed unused Test Points from Schematic
Parts:
- removed TP1, TP15, TP17, TP18, TP19, TP2, TP20, TP21, TP23, TP24, TP25, TP26, TP27, TP28, TP29, TP3, TP30, TP32, TP33, TP34, TP35, TP36, TP37, TP38, TP39, TP4, TP40, TP41, TP42, TP43, TP44, TP45, TP46, TP47, TP48, TP49, TP50, TP51, TP52, TP53, TP54, TP55, TP56, TP57, TP58, TP59, TP60, TP61, TP62, TP63, TP64, TP65, TP66, TP67, TP68, TP69, TP70, TP71, TP72, TP73, TP74, TP75, TP76, TP77, TP78, TP79, TP80, TP81, TP82, TP83, TP84: TestPoint, TestPoint:TestPoint_Pad_1.0x1.0mm, symbol Connector:TestPoint
- added R7: 100, Resistor_SMD:R_0603_1608Metric, symbol Device:R
- TP10: value TestPoint -> TST
- TP11: value TestPoint -> VDDOUT
- TP12: value TestPoint -> WKUP0
- TP13: value TestPoint -> XIN32
- TP14: value TestPoint -> XOUT32
- TP15: value TestPoint -> nRST
- TP16: value TestPoint -> XOUT
- TP22: value TestPoint -> CLK_FROM_SAM
- TP5: value TestPoint -> ERASE
- TP6: value TestPoint -> FWUP
- TP7: value TestPoint -> JTAGSEL
- TP8: value TestPoint -> SHDN
- TP9: value TestPoint -> VDDLCD
Connections:
- net VCC1.2: now also R7.1; no longer C4.1, C5.1, U1.53 (VDDPLL)
- new net: C4.1, C5.1, R7.2, U1.53 (VDDPLL)
- no-connect marks 28 -> 88
Other:
- moved on the sheet: C4, C5

Commit message: Changed processor footprint to have pad spacing of 0.22mm so black solder mask will bridge.
Parts:
- U1: footprint Package_QFP:TQFP-100_14x14mm_P0.5mm -> RECESSIM-CW312T-SAM4C32:TQFP-100_14x14mm_P0.5mm_W0.28mm
Changed lines of the file:
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@@
 			)
 		)
-		(property "Footprint" "Package_QFP:TQFP-100_14x14mm_P0.5mm"
+		(property "Footprint" "RECESSIM-CW312T-SAM4C32:TQFP-100_14x14mm_P0.5mm_W0.28mm"
 			(at 82.296 147.066 0)
 			(effects

Commit message: Fixed TX/RX UART pin locations, updated PCB and regenerated gerbers
Connections:
- net GPIO1_TX: now also U1.45 (PB5); no longer U1.69 (PA10/PGMM2)
- net GPIO2_RX: now also U1.43 (PB4); no longer U1.68 (PA9/PGMM1)
Other:
- title: (none) -> SAM4C32C Target Board
Changed lines of the file:
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@@
 	(generator_version "8.0")
 	(paper "A4")
+	(title_block
+		(title "SAM4C32C Target Board")
+		(rev "2")
+	)
 	(junction
 		(at 59.69 184.15)
@@
 	)
 	(no_connect
-		(at 182.88 49.53)
+		(at 105.41 35.56)
 	)
 	(no_connect
@@
 	)
 	(no_connect
+		(at 102.87 35.56)
+	)
+	(no_connect
 		(at 273.05 110.49)
 	)
@@
 	)
 	(no_connect
-		(at 182.88 46.99)
-	)
-	(no_connect
 		(at 273.05 102.87)
 	)
@@
 	(wire
 		(pts
-			(xy 102.87 21.59) (xy 102.87 35.56)
-		)
-		(stroke
-			(width 0)
-			(type default)
-		)
-	)
-	(wire
-		(pts
 			(xy 207.01 59.69) (xy 231.14 59.69)
 		)
@@
 	(wire
 		(pts
+			(xy 182.88 46.99) (xy 196.85 46.99)
+		)
+		(stroke
+			(width 0)
+			(type default)
+		)
+	)
+	(wire
+		(pts
 			(xy 72.39 184.15) (xy 77.47 184.15)
 		)
@@
 	(wire
 		(pts
-			(xy 105.41 21.59) (xy 105.41 35.56)
-		)
-		(stroke
-			(width 0)
-			(type default)
-		)
-	)
-	(wire
-		(pts
 			(xy 116.84 165.1) (xy 116.84 166.37)
 		)
@@
 		(pts
 			(xy 115.57 190.5) (xy 116.84 190.5)
+		)
+		(stroke
+			(width 0)
+			(type default)
+		)
+	)
+	(wire
+		(pts
+			(xy 182.88 49.53) (xy 196.85 49.53)
 		)
 		(stroke
@@
 	)
 	(label "GPIO2_RX"
-		(at 102.87 33.02 90)
+		(at 185.42 46.99 0)
 		(fields_autoplaced yes)
 		(effects
@@
 	)
 	(label "GPIO1_TX"
-		(at 105.41 33.02 90)
-		(fields_autoplaced yes)
-		(effects
+		(at 185.42 49.53 0)
+		(fields_autoplaced yes)
+		(effects
